File: PCBDesign01.sch (EAGLE design)
At the start: 87 parts, among them IC1 TESEO-LIV3R, J1 5051102491, U1 TPS71913-28DRVR, U3 CD40109BPWR, U4 MCP23017T-E/SO

Commit message: ready for pcb review
Parts:
- removed U$14, U$19, U$20, U$22: TESTPOINT, Test Point:TESTPOINT
- LEDG: value 60 -> 60.4
- LEDR: value 80 -> 80.6
- R3: value 86.6 -> 80.6
Connections:
- net GND: no longer U$14.0, U$19.0, U$20.0, U$22.0
- net LED_B: now also U4.GPA0; no longer U4.GPA2
- net LED_R: now also U4.GPA2; no longer U4.GPA0
Changed lines of the file:
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@@
 <part name="D2" library="CLX6F-FKC-CKNNQDGBB7A363" deviceset="CLX6F-FKC-CKNNQDGBB7A363" device=""/>
 <part name="J1" library="5051102491" deviceset="5051102491" device=""/>
-<part name="LEDR" library="Resistor" library_urn="urn:adsk.eagle:library:16378527" deviceset="R-US" device="CHIP-0805(2012-METRIC)" package3d_urn="urn:adsk.eagle:package:16378559/2" technology="_" value="80"/>
-<part name="LEDG" library="Resistor" library_urn="urn:adsk.eagle:library:16378527" deviceset="R-US" device="CHIP-0805(2012-METRIC)" package3d_urn="urn:adsk.eagle:package:16378559/2" technology="_" value="60"/>
+<part name="LEDR" library="Resistor" library_urn="urn:adsk.eagle:library:16378527" deviceset="R-US" device="CHIP-0805(2012-METRIC)" package3d_urn="urn:adsk.eagle:package:16378559/2" technology="_" value="80.6"/>
+<part name="LEDG" library="Resistor" library_urn="urn:adsk.eagle:library:16378527" deviceset="R-US" device="CHIP-0805(2012-METRIC)" package3d_urn="urn:adsk.eagle:package:16378559/2" technology="_" value="60.4"/>
 <part name="LEDB" library="Resistor" library_urn="urn:adsk.eagle:library:16378527" deviceset="R-US" device="CHIP-0805(2012-METRIC)" package3d_urn="urn:adsk.eagle:package:16378559/2" technology="_" value="30"/>
-<part name="R3" library="Resistor" library_urn="urn:adsk.eagle:library:16378527" deviceset="R-US" device="CHIP-0805(2012-METRIC)" package3d_urn="urn:adsk.eagle:package:16378559/2" technology="_" value="86.6"/>
+<part name="R3" library="Resistor" library_urn="urn:adsk.eagle:library:16378527" deviceset="R-US" device="CHIP-0805(2012-METRIC)" package3d_urn="urn:adsk.eagle:package:16378559/2" technology="_" value="80.6"/>
 <part name="SUPPLY1" library="supply2" library_urn="urn:adsk.eagle:library:372" deviceset="GND" device=""/>
 <part name="SUPPLY6" library="supply2" library_urn="urn:adsk.eagle:library:372" deviceset="GND" device=""/>
@@
 <part name="U$12" library="Test Point" deviceset="TESTPOINT" device=""/>
 <part name="U$13" library="Test Point" deviceset="TESTPOINT" device=""/>
-<part name="U$14" library="Test Point" deviceset="TESTPOINT" device=""/>
 <part name="U$15" library="Test Point" deviceset="TESTPOINT" device=""/>
 <part name="U$16" library="Test Point" deviceset="TESTPOINT" device=""/>
 <part name="U$17" library="Test Point" deviceset="TESTPOINT" device=""/>
 <part name="U$18" library="Test Point" deviceset="TESTPOINT" device=""/>
-<part name="U$19" library="Test Point" deviceset="TESTPOINT" device=""/>
-<part name="U$20" library="Test Point" deviceset="TESTPOINT" device=""/>
 <part name="U$21" library="Test Point" deviceset="TESTPOINT" device=""/>
-<part name="U$22" library="Test Point" deviceset="TESTPOINT" device=""/>
 <part name="U$23" library="Test Point" deviceset="TESTPOINT" device=""/>
 <part name="U$24" library="Test Point" deviceset="TESTPOINT" device=""/>
@@
 <instance part="LEDR" gate="G$1" x="0" y="-101.6" smashed="yes" rot="R90">
 <attribute name="NAME" x="-1.4986" y="-105.41" size="1.778" layer="95" rot="R90"/>
-<attribute name="VALUE" x="3.302" y="-102.87" size="1.778" layer="96" rot="R90"/>
+<attribute name="VALUE" x="3.048" y="-104.14" size="1.778" layer="96" rot="R90"/>
 </instance>
 <instance part="LEDG" gate="G$1" x="7.62" y="-101.6" smashed="yes" rot="R90">
 <attribute name="NAME" x="6.1214" y="-105.41" size="1.778" layer="95" rot="R90"/>
-<attribute name="VALUE" x="10.922" y="-102.87" size="1.778" layer="96" rot="R90"/>
+<attribute name="VALUE" x="10.922" y="-104.14" size="1.778" layer="96" rot="R90"/>
 </instance>
 <instance part="LEDB" gate="G$1" x="15.24" y="-101.6" smashed="yes" rot="R90">
@@
 <instance part="U$12" gate="A" x="154.94" y="2.54" smashed="yes"/>
 <instance part="U$13" gate="A" x="-101.6" y="83.82" smashed="yes"/>
-<instance part="U$14" gate="A" x="-78.74" y="91.44" smashed="yes" rot="R180"/>
 <instance part="U$15" gate="A" x="-86.36" y="83.82" smashed="yes"/>
 <instance part="U$16" gate="A" x="-93.98" y="83.82" smashed="yes"/>
 <instance part="U$17" gate="A" x="-71.12" y="83.82" smashed="yes"/>
 <instance part="U$18" gate="A" x="-78.74" y="83.82" smashed="yes"/>
-<instance part="U$19" gate="A" x="-71.12" y="91.44" smashed="yes" rot="R180"/>
-<instance part="U$20" gate="A" x="-93.98" y="91.44" smashed="yes" rot="R180"/>
-<instance part="U$21" gate="A" x="-86.36" y="91.44" smashed="yes" rot="R180"/>
-<instance part="U$22" gate="A" x="-101.6" y="91.44" smashed="yes" rot="R180"/>
+<instance part="U$21" gate="A" x="-101.6" y="91.44" smashed="yes" rot="R180"/>
 <instance part="U$23" gate="A" x="106.68" y="111.76" smashed="yes"/>
 <instance part="U$24" gate="A" x="-157.48" y="-129.54" smashed="yes"/>
@@
 <instance part="U$26" gate="A" x="-149.86" y="-129.54" smashed="yes"/>
 <instance part="U$27" gate="A" x="-134.62" y="-129.54" smashed="yes"/>
-<instance part="SUPPLY16" gate="GND" x="-86.36" y="101.6" smashed="yes" rot="R180">
-<attribute name="VALUE" x="-84.455" y="104.775" size="1.778" layer="96" rot="R180"/>
+<instance part="SUPPLY16" gate="GND" x="-101.6" y="101.6" smashed="yes" rot="R180">
+<attribute name="VALUE" x="-99.695" y="104.775" size="1.778" layer="96" rot="R180"/>
 </instance>
 <instance part="U$9" gate="A" x="114.3" y="111.76" smashed="yes"/>
@@
 </segment>
 <segment>
-<pinref part="U$19" gate="A" pin="0"/>
-<pinref part="U$22" gate="A" pin="0"/>
-<wire x1="-71.12" y1="99.06" x2="-78.74" y2="99.06" width="0.1524" layer="91"/>
-<pinref part="U$14" gate="A" pin="0"/>
-<wire x1="-78.74" y1="99.06" x2="-86.36" y2="99.06" width="0.1524" layer="91"/>
-<junction x="-78.74" y="99.06"/>
-<pinref part="U$20" gate="A" pin="0"/>
-<wire x1="-86.36" y1="99.06" x2="-93.98" y2="99.06" width="0.1524" layer="91"/>
-<wire x1="-93.98" y1="99.06" x2="-101.6" y2="99.06" width="0.1524" layer="91"/>
-<junction x="-93.98" y="99.06"/>
 <pinref part="U$21" gate="A" pin="0"/>
-<junction x="-86.36" y="99.06"/>
 <pinref part="SUPPLY16" gate="GND" pin="GND"/>
 </segment>
@@
 </segment>
 <segment>
-<wire x1="-17.78" y1="-25.4" x2="-20.32" y2="-25.4" width="0.1524" layer="91"/>
-<label x="-17.78" y="-25.4" size="1.778" layer="95" xref="yes"/>
-<pinref part="U4" gate="G$1" pin="GPA0"/>
+<wire x1="-17.78" y1="-30.48" x2="-20.32" y2="-30.48" width="0.1524" layer="91"/>
+<label x="-17.78" y="-30.48" size="1.778" layer="95" xref="yes"/>
+<pinref part="U4" gate="G$1" pin="GPA2"/>
 </segment>
 </net>
@@
 </segment>
 <segment>
-<wire x1="-17.78" y1="-30.48" x2="-20.32" y2="-30.48" width="0.1524" layer="91"/>
-<label x="-17.78" y="-30.48" size="1.778" layer="95" xref="yes"/>
-<pinref part="U4" gate="G$1" pin="GPA2"/>
-</segment>
-</net>
+<wire x1="-17.78" y1="-25.4" x2="-20.32" y2="-25.4" width="0.1524" layer="91"/>
+<label x="-17.78" y="-25.4" size="1.778" layer="95" xref="yes"/>
+<pinref part="U4" gate="G$1" pin="GPA0"/>
+</segment>
+</net>

Commit message: add magnetometer
Parts:
- added C24, C25, C26, C27: 0.1uF, Capacitor:C_CHIP-0805(2012-METRIC)
- added C28: 4.7uF, Capacitor:C_CHIP-0805(2012-METRIC)
- added R19: 10k, Resistor:R-US_CHIP-0805(2012-METRIC)
- added U2: FXOS8700CQR1, FXOS8700CQR1 Magnetometer:FXOS8700CQR1
Connections:
- new net N$18: C25.1, U2.BYP
- new net N$5: C26.1, U2.CRST
- net 3.3V: now also C24.2, C27.1, C28.1, R19.1, U2.VDD, U2.VDDIO
- net GND: now also C24.1, C25.2, C26.2, C27.2, C28.2, U2.GND, U2.GND_2, U2.RESERVED, U2.RESERVED_2, U2.RST, U2.SA0/MISO, U2.SA1/CS_B
- net I2C_SCL: now also R19.2, U2.SCL/SCLK
- net I2C_SDA: now also U2.SDA/MOSI
Other:
- note added: "I2C Address: 0011110"
- note added: "Magnetometer"
- moved on the sheet: BACK-LEFT, BACK-RIGHT, C10, C12, C13, C14, C15, C17, C18, C19, C20, C21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
