File: PCBDesign01.brd (EAGLE design)
At the start: 101.6 x 101.6 mm, 90 parts, among them IC1 TESEO-LIV3R, J1 5051102491, U1 TPS71913-28DRVR, U2 FXOS8700CQR1, U3 CD40109BPWR, U4 MCP23017T-E/SO

Commit message: verification
Parts:
- moved C23 3.23 mm to (11.7, -19.8)
- moved U$4 2.54 mm to (8.46, -24.5), turned to 180 degrees
Connections:
- net GND: now also U1.8, U1.9
Routing:
- net I2C_SDA: track 139.0 -> 148.7 mm
- net GND: track 164.7 -> 171.4 mm, vias 77 -> 150
- net ANT: track 5.79 -> 4.18 mm
- net VCC_RF: track 9.32 -> 7.95 mm
- net I2C_SCL: track 140.2 -> 139.3 mm
- net N$18: track 5.75 -> 6.64 mm
- net SD_DAT0: track 181.0 -> 180.2 mm
- net VBAT: track 52.8 -> 52.2 mm
- added copper zone on layer 1, net GND

Commit message: names
Parts:
- added U$14, U$19, U$2, U$20: TESTPOINT, Test Point:TESTPOINT
- moved C19 99.2 mm to (69.2, 84.6)
- moved C5 99.2 mm to (59.8, 74.2)
- moved A1 99.2 mm to (97.9, 100.7)
- moved BACK-LEFT 99.2 mm to (125.9, 30.1)
- moved BACK-RIGHT 99.2 mm to (126.6, 121.8)
- moved BUZZER 99.2 mm to (102.6, 60.9)
- moved C1 99.2 mm to (86.7, 70.6)
- moved C10 99.2 mm to (59.8, 81.6)
- moved C11 99.2 mm to (112.4, 108.8)
- moved C12 99.2 mm to (59.7, 109.7)
- moved C13 99.2 mm to (52.7, 107.7)
- moved C14 99.2 mm to (63.7, 109.7)
- moved C15 99.2 mm to (47.3, 107.8)
- moved C16 99.2 mm to (90.2, 57.5)
- moved C17 99.2 mm to (94.7, 117.2)
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Connections:
- new net GPIO_A6: U$2.0, U4.27
- new net GPIO_A7: U$19.0, U4.28
- new net GPIO_B6: U$14.0, U4.7
- new net GPIO_B7: U$20.0, U4.8
Routing:
- net GPIO_A6: track 0.00 -> 50.6 mm, vias 0 -> 2
- net GPIO_B7: track 0.00 -> 47.0 mm, vias 0 -> 3
- net GPIO_B6: track 0.00 -> 45.2 mm, vias 0 -> 3
- net GPIO_A7: track 0.00 -> 44.1 mm, vias 0 -> 2
- net ESC_BL_OUT: track 125.3 -> 115.3 mm
- net ESC_BR_OUT: track 59.4 -> 51.4 mm
- net ESC_FL_OUT: track 216.1 -> 210.7 mm
- net ESC_FR_OUT: track 126.8 -> 121.5 mm
- net GND: track 171.4 -> 174.3 mm, vias 150 -> 152
- net ESC_FR: track 74.2 -> 75.9 mm
- net 5V: track 309.1 -> 307.6 mm
Other:
- board text added: "+"
- board text added: "-"
- board text added: "2020 POWER UP FIG QUADCOPTER"
- board text added: "A6"
- board text added: "A7"
- board text added: "Adeel Rehman Alec Neiman Allen Jiang Andy Ly Jason Math Jeffrey Liu Lauren Head Masaad Khan Ryan McSweeney"
- board text added: "B6"
- board text added: "B7"
- board text added: "Back Left"
- board text added: "Back Right"
- board text added: "Front Left"
- board text added: "Front Right"
