File: PCBDesign01.brd (EAGLE design)
At the start: 101.6 x 101.6 mm, 94 parts, among them IC1 TESEO-LIV3R, J1 5051102491, U1 TPS71913-28DRVR, U2 FXOS8700CQR1, U3 CD40109BPWR, U4 MCP23017T-E/SO

Commit message: minor adjustments
Parts:
- J1: value 5051102491 -> 5051102491ACTUAL; device 5051102491:5051102491 -> 5051102491:687124149022
- moved J1 1.69 mm to (52.4, 77.3)
Connections:
- net GND: now also J1.Z1, J1.Z2; no longer J1.25, J1.26
Routing:
- net DVP_VSYNC: track 76.6 -> 79.7 mm
- net DVP_HREF: track 54.4 -> 56.9 mm
- net GND: track 174.3 -> 176.3 mm
- net DVP_Y5: track 57.2 -> 58.9 mm
- net CAM_RESET: track 19.9 -> 21.1 mm
- net DVP_Y3: track 5.47 -> 6.61 mm
- net 1.3V: track 53.9 -> 55.0 mm
- net CAM_I2C_SCL: track 85.9 -> 86.9 mm
- net 3.3V: track 160.4 -> 161.4 mm
- net XMCLK: track 62.7 -> 63.7 mm
- net DVP_Y7: track 5.61 -> 6.63 mm
- net DVP_Y4: track 6.24 -> 7.26 mm
- net DVP_Y9: track 80.9 -> 81.9 mm
- net DVP_Y6: track 49.0 -> 50.0 mm
- net DVP_Y2: track 56.8 -> 57.8 mm
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
Commit message: final?
Parts:
- removed U1: TPS71913-28DRVR, TPS71913-28DRVR:DRV6_1P6X1
- added C29: 1uF, Capacitor:CAPC2012X110
- added U5: MIC5504-2.8YM5-TR, MIC5504_2.8YM5:SOT95P280X145-5N
- added U6: MIC5365-1.3YC5-TRSC-70_C5_MCH-M, MIC5365_1.3YC5:SC-70_C5_MCH-M
- moved C7 5.13 mm to (35.0, 113.5)
- moved C6 4.60 mm to (41.5, 111.0), turned to 270 degrees
- moved C8 3.85 mm to (34.9, 109.5)
Connections:
- net 1.3V: now also U6.5; no longer U1.1
- net 2.8V: now also U5.5; no longer U1.3
- net 3.3V: now also C29.1, U5.1, U5.3, U6.1, U6.3; no longer U1.2, U1.4, U1.6
- net GND: now also C29.2, U5.2, U6.2; no longer U1.5, U1.7, U1.8, U1.9
Routing:
- net 2.8V: track 51.1 -> 60.0 mm
- net GND: track 176.3 -> 168.0 mm, vias 152 -> 150
- net 1.3V: track 55.0 -> 52.1 mm
- net 3.3V: track 161.4 -> 163.3 mm
Other:
- board text added: "Class of 2023 Zoom University"

Commit message: final.
Routing:
- net 3.3V: track 163.3 -> 172.4 mm, vias 35 -> 37
- net I2C_SCL: track 139.3 -> 134.8 mm
- net GND: track 168.0 -> 172.3 mm, vias 150 -> 152
Changed lines of the file:
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@@
 <wire x1="85.011996875" y1="76.193759375" x2="85.253971875" y2="75.951784375" width="0.1524" layer="1"/>
 <via x="85.253971875" y="75.951784375" extent="1-16" drill="0.35"/>
-<wire x1="79.0762" y1="76.993759375" x2="78.059365625" y2="76.993759375" width="0.1524" layer="1"/>
-<wire x1="78.059365625" y1="76.993759375" x2="78.051628125" y2="77.001496875" width="0.1524" layer="1"/>
-<via x="78.051628125" y="77.001496875" extent="1-16" drill="0.35"/>
+<wire x1="79.0762" y1="76.993759375" x2="78.5553875" y2="76.993759375" width="0.1524" layer="1"/>
+<wire x1="78.5553875" y1="76.993759375" x2="78.065175" y2="77.483971875" width="0.1524" layer="1"/>
+<via x="78.065175" y="77.483971875" extent="1-16" drill="0.35"/>
 <wire x1="70.4962" y1="88.783759375" x2="70.4962" y2="86.806040625" width="0.1524" layer="1"/>
 <wire x1="70.4962" y1="86.806040625" x2="70.9009125" y2="86.401328125" width="0.1524" layer="1"/>
@@
 <contactref element="C29" pad="2"/>
 <contactref element="C8" pad="2"/>
+<polygon width="0.1524" layer="16" pour="cutout">
+<vertex x="108" y="69.5"/>
+<vertex x="109.5" y="69.5"/>
+<vertex x="109.5" y="68"/>
+<vertex x="108" y="68"/>
+</polygon>
+<via x="105.924290625" y="68.529953125" extent="1-16" drill="0.35"/>
+<wire x1="107.131690625" y1="69.2088" x2="107.1314875" y2="69.208596875" width="0.1524" layer="16"/>
+<wire x1="107.1314875" y1="69.208596875" x2="106.405803125" y2="69.208596875" width="0.1524" layer="16"/>
+<wire x1="106.405803125" y1="69.208596875" x2="105.923828125" y2="68.726621875" width="0.1524" layer="16"/>
+<wire x1="105.924290625" y1="68.529953125" x2="105.923828125" y2="68.530415625" width="0.1524" layer="16"/>
+<wire x1="105.923828125" y1="68.726621875" x2="105.923828125" y2="68.530415625" width="0.1524" layer="16"/>
+<wire x1="105.924290625" y1="68.529953125" x2="104.5" y2="69.95424375" width="0.1524" layer="1"/>
+<wire x1="104.5" y1="69.95424375" x2="104.5" y2="70.5" width="0.1524" layer="1"/>
+<via x="104.5" y="70.5" extent="1-16" drill="0.35"/>
 </signal>
 <signal name="3.3V">
@@
 <wire x1="72.317678125" y1="67.616296875" x2="74.7446375" y2="70.04325625" width="0.1524" layer="1"/>
 <wire x1="82.461140625" y1="69.70064375" x2="82.118528125" y2="70.04325625" width="0.1524" layer="1"/>
-<wire x1="82.118528125" y1="70.04325625" x2="74.7446375" y2="70.04325625" width="0.1524" layer="1"/>
+<wire x1="82.118528125" y1="70.04325625" x2="76" y2="70.04325625" width="0.1524" layer="1"/>
+<wire x1="76" y1="70.04325625" x2="74.7446375" y2="70.04325625" width="0.1524" layer="1"/>
 <wire x1="84.025196875" y1="75.37701875" x2="84.025196875" y2="71.784359375" width="0.1524" layer="16"/>
 <wire x1="84.025196875" y1="71.784359375" x2="82.461140625" y2="70.220303125" width="0.1524" layer="16"/>
@@
 <wire x1="41.5" y1="111.8754" x2="41.5" y2="113" width="0.1524" layer="16"/>
 <via x="41.5" y="113" extent="1-16" drill="0.35"/>
+<polygon width="0.1524" layer="1" pour="cutout">
+<vertex x="79.5" y="77.5"/>
+<vertex x="79.5" y="75.269690625"/>
+<vertex x="79.6263625" y="75.143328125"/>
+<vertex x="81.85865" y="75.143328125"/>
+<vertex x="81.997415625" y="75.28209375"/>
+<vertex x="81.997415625" y="77.4902375"/>
+<vertex x="81.89485" y="77.592803125"/>
+<vertex x="79.592803125" y="77.592803125"/>
+</polygon>
+<wire x1="79.0762" y1="76.193759375" x2="78.332603125" y2="76.193759375" width="0.1524" layer="1"/>
+<wire x1="78.332603125" y1="76.193759375" x2="78.0263625" y2="76.5" width="0.1524" layer="1"/>
+<via x="78.0263625" y="76.5" extent="1-16" drill="0.35"/>
+<wire x1="78.0263625" y1="76.5" x2="78.0263625" y2="73.5263625" width="0.1524" layer="16"/>
+<wire x1="75.80474375" y1="71.30474375" x2="75.80474375" y2="69.81445625" width="0.1524" layer="16"/>
+<via x="75.80474375" y="69.81445625" extent="1-16" drill="0.35"/>
+<wire x1="75.80474375" y1="69.81445625" x2="75.80474375" y2="69.848" width="0.1524" layer="1"/>
+<wire x1="75.80474375" y1="69.848" x2="76" y2="70.04325625" width="0.1524" layer="1"/>
+<wire x1="78.0263625" y1="73.5263625" x2="75.80474375" y2="71.30474375" width="0.1524" layer="16"/>
 </signal>
 <signal name="5V">
@@
 <wire x1="107.9912" y1="94.9388" x2="106.6812" y2="94.9388" width="0.1524" layer="16"/>
 <wire x1="79.0762" y1="75.793759375" x2="79.072834375" y2="75.79039375" width="0.1524" layer="1"/>
-<wire x1="79.072834375" y1="75.79039375" x2="78.5081125" y2="75.79039375" width="0.1524" layer="1"/>
-<wire x1="78.5081125" y1="75.79039375" x2="73.0362" y2="81.26230625" width="0.1524" layer="1"/>
 <wire x1="73.0362" y1="81.26230625" x2="73.0362" y2="88.783759375" width="0.1524" layer="1"/>
 <wire x1="48.9725125" y1="59.2088" x2="43.695425" y2="53.9317125" width="0.1524" layer="1"/>
@@
 <wire x1="91.9962125" y1="80.468003125" x2="92.755415625" y2="79.7088" width="0.1524" layer="1"/>
 <wire x1="78.597103125" y1="80.468003125" x2="91.9962125" y2="80.468003125" width="0.1524" layer="1"/>
+<wire x1="75.079134375" y1="78.239815625" x2="75.079134375" y2="79.219371875" width="0.1524" layer="1"/>
+<wire x1="75.079134375" y1="79.219371875" x2="73.0362" y2="81.26230625" width="0.1524" layer="1"/>
 </signal>
 <signal name="ANT">
@@
 <contactref element="U2" pad="2"/>
 <wire x1="108.2212" y1="70.295875" x2="108.2212" y2="71.203671875" width="0.1524" layer="16"/>
-<wire x1="108.2212" y1="71.203671875" x2="107.811340625" y2="71.61353125" width="0.1524" layer="16"/>
-<wire x1="107.811340625" y1="71.61353125" x2="107.00833125" y2="71.61353125" width="0.1524" layer="16"/>
-<wire x1="107.00833125" y1="71.61353125" x2="103.99484375" y2="68.60004375" width="0.1524" layer="16"/>
+<wire x1="108.2212" y1="71.203671875" x2="107.99025" y2="71.434621875" width="0.1524" layer="16"/>
+<wire x1="107.99025" y1="71.434621875" x2="106.829421875" y2="71.434621875" width="0.1524" layer="16"/>
+<wire x1="106.829421875" y1="71.434621875" x2="103.99484375" y2="68.60004375" width="0.1524" layer="16"/>
 <wire x1="103.99484375" y1="68.60004375" x2="103.9097125" y2="68.60004375" width="0.1524" layer="16"/>
 </signal>
